File: PCB/Smedby Charger prot.brd (EAGLE design)
At the start: 100 x 80 mm, 90 parts, among them IC2 TLC274D, Q1 BD140, Q10 BD139, Q2 TIP41C, Q3 BD139, Q4 IRF9530, Q7 BD139, T1 BC547, T2 TIP32

Commit message: .svn stuff removesd
Parts:
- R10: value 380 -> 1k
Changed lines of the file:
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@@
 <?xml version="1.0" encoding="utf-8"?>
 <!DOCTYPE eagle SYSTEM "eagle.dtd">
-<eagle version="6.4">
+<eagle version="6.5.0">
 <drawing>
 <settings>
@@
 <element name="Q3" library="transistor-power" package="TO126AV" value="BD139" x="-20.32" y="-99.06"/>
 <element name="Q4" library="transistor-fet" package="TO220" value="IRF9530" x="-43.18" y="-121.92"/>
-<element name="R10" library="rcl" package="P0613V" value="380" x="-15.24" y="-185.42"/>
+<element name="R10" library="rcl" package="P0613V" value="1k" x="-15.24" y="-185.42"/>
 <element name="C11" library="rcl" package="E7,5-18" value="1000u" x="-39.37" y="-165.1"/>
 <element name="C13" library="rcl" package="C050-024X044" value="100n" x="-24.13" y="-185.42"/>

Commit message: Uppdated PCB
Parts:
- removed C11: 1000u, rcl:E7,5-18
- removed C13: 100n, rcl:C050-024X044
- removed D4: 1N5400, diode:DO201-15
- removed L2: 150uH, rcl:TJ4-U1
- added C6, C7: 100u, rcl:E2,5-5
- added Q5: IRF540, transistor-power:TO220BV
- added R35: 100, rcl:P0613V
- added U1: IR2103, irf-2:DIL08
- D1: value 1N5400 -> 1N4148DO35-7; device diode:DO201-15 -> diode:DO35-7
- moved T2 219.5 mm to (83.8, 31.8), turned to 270 degrees
- moved Q4 189.7 mm to (83.8, 19.1), turned to 270 degrees
- moved D1 62.3 mm to (-41.9, -241.3)
Connections:
- removed net B+1: D4.C
- removed net N$21: D14.C, L1.1, Q4.2
- new net CHOPEDPOWER: D14.C, L1.1, Q1.C, Q4.2, Q5.S, T2.2
- new net VB: C7.+, D1.C, U1.8
- new net VCC: C6.+, D1.A, U1.1
- net CHARGEPWM: now also R3.1, U1.2
- net GND: now also C6.-, U1.3, U1.4; no longer C11.-, C13.2, D1.A
- net N$2: now also C7.-, U1.6; no longer D1.C, L2.1, Q1.C, T2.2
- net N$20: now also R35.1, U1.7; no longer C11.+, C13.1, D4.A, L2.2
- net N$4: now also Q5.G, R35.2; no longer R3.1
- net V+: now also Q5.D
Changed lines of the file:
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@@
 <layer number="97" name="Info" color="7" fill="1" visible="no" active="no"/>
 <layer number="98" name="Guide" color="6" fill="1" visible="no" active="no"/>
+<layer number="100" name="Muster" color="7" fill="1" visible="no" active="no"/>
+<layer number="250" name="Descript" color="3" fill="1" visible="no" active="no"/>
+<layer number="251" name="SMDround" color="12" fill="11" visible="no" active="no"/>
 </layers>
 <board>
@@
 <element name="R34" library="rcl" package="0207/2V" value="1k" x="-17.78" y="-128.27"/>
 <element name="Q3" library="transistor-power" package="TO126AV" value="BD139" x="-20.32" y="-99.06"/>
-<element name="Q4" library="transistor-fet" package="TO220" value="IRF9530" x="-43.18" y="-121.92"/>
+<element name="Q4" library="transistor-fet" package="TO220" value="IRF9530" x="83.82" y="19.05" rot="R270"/>
 <element name="R10" library="rcl" package="P0613V" value="1k" x="-15.24" y="-185.42"/>
-<element name="C11" library="rcl" package="E7,5-18" value="1000u" x="-39.37" y="-165.1"/>
-<element name="C13" library="rcl" package="C050-024X044" value="100n" x="-24.13" y="-185.42"/>
-<element name="L2" library="rcl" package="TJ4-U1" value="150uH" x="-31.75" y="-143.51"/>
-<element name="D1" library="diode" package="DO201-15" value="1N5400" x="-38.1" y="-179.07"/>
-<element name="D4" library="diode" package="DO201-15" value="1N5400" x="-38.1" y="-187.96"/>
 <element name="R2" library="rcl" package="0207/2V" value="10k" x="-45.72" y="-194.31"/>
 <element name="T1" library="transistor" package="TO92" value="BC547" x="-33.02" y="-194.31"/>
 <element name="R3" library="rcl" package="0207/2V" value="1k" x="-39.37" y="-194.31"/>
-<element name="T2" library="transistor" package="TO220" value="TIP32" x="-43.18" y="-147.32"/>
+<element name="T2" library="transistor" package="TO220" value="TIP32" x="83.82" y="31.75" rot="R270"/>
 <element name="Q1" library="transistor-power" package="TO126AV" value="BD140" x="-43.18" y="-198.12"/>
+<element name="U1" library="irf-2" package="DIL08" value="IR2103" x="-40.64" y="-210.82"/>
+<element name="Q5" library="transistor-power" package="TO220BV" value="IRF540" x="100.33" y="49.53" rot="R270"/>
+<element name="C6" library="rcl" package="E2,5-5" value="100u" x="-45.72" y="-228.6"/>
+<element name="C7" library="rcl" package="E2,5-5" value="100u" x="-45.72" y="-234.95"/>
+<element name="D1" library="diode" package="DO35-7" value="1N4148DO35-7" x="-41.91" y="-241.3"/>
+<element name="R35" library="rcl" package="P0613V" value="100" x="-43.18" y="-247.65"/>
 </elements>
 <signals>
@@
 <contactref element="Q3" pad="E"/>
 <contactref element="R32" pad="1"/>
-<contactref element="C11" pad="-"/>
-<contactref element="C13" pad="2"/>
-<contactref element="D1" pad="A"/>
 <contactref element="T1" pad="1"/>
-<wire x1="-21.59" y1="-185.42" x2="-31.75" y2="-194.31" width="0" layer="19" extent="1-1"/>
-<wire x1="-30.48" y1="-179.07" x2="-21.59" y2="-185.42" width="0" layer="19" extent="1-1"/>
-<wire x1="-35.56" y1="-165.1" x2="-30.48" y2="-179.07" width="0" layer="19" extent="1-1"/>
-<wire x1="-33.02" y1="-128.27" x2="-35.56" y2="-165.1" width="0" layer="19" extent="1-1"/>
+<contactref element="U1" pad="4"/>
+<contactref element="C6" pad="-"/>
+<contactref element="U1" pad="3"/>
+<wire x1="-36.83" y1="-214.63" x2="-39.37" y2="-214.63" width="0" layer="19" extent="1-1"/>
+<wire x1="-44.45" y1="-228.6" x2="-39.37" y2="-214.63" width="0" layer="19" extent="1-1"/>
+<wire x1="-31.75" y1="-194.31" x2="-36.83" y2="-214.63" width="0" layer="19" extent="1-1"/>
+<wire x1="-33.02" y1="-128.27" x2="-31.75" y2="-194.31" width="0" layer="19" extent="1-1"/>
 <wire x1="-17.78" y1="-113.03" x2="-33.02" y2="-128.27" width="0" layer="19" extent="1-1"/>
 <wire x1="-8.89" y1="-119.38" x2="-17.78" y2="-113.03" width="0" layer="19" extent="1-1"/>
@@
 <contactref element="R2" pad="1"/>
 <contactref element="T2" pad="3"/>
-<wire x1="-40.64" y1="-153.67" x2="-46.99" y2="-194.31" width="0" layer="19" extent="1-1"/>
-<wire x1="-40.64" y1="-128.27" x2="-40.64" y2="-153.67" width="0" layer="19" extent="1-1"/>
-<wire x1="-25.4" y1="-128.27" x2="-40.64" y2="-128.27" width="0" layer="19" extent="1-1"/>
+<contactref element="Q5" pad="D"/>
+<wire x1="97.79" y1="49.53" x2="-46.99" y2="-194.31" width="0" layer="19" extent="1-1"/>
+<wire x1="77.47" y1="29.21" x2="-46.99" y2="-194.31" width="0" layer="19" extent="1-1"/>
+<wire x1="77.47" y1="16.51" x2="77.47" y2="29.21" width="0" layer="19" extent="1-1"/>
+<wire x1="-25.4" y1="-128.27" x2="77.47" y2="16.51" width="0" layer="19" extent="1-1"/>
 <wire x1="-31.75" y1="-72.39" x2="-25.4" y2="-128.27" width="0" layer="19" extent="1-1"/>
 <wire x1="29.21" y1="11.37" x2="-31.75" y2="-72.39" width="0" layer="19" extent="1-1"/>
@@
 <contactref element="MODUL1" pad="J1.6"/>
 <contactref element="R34" pad="1"/>
+<contactref element="R3" pad="1"/>
+<contactref element="U1" pad="2"/>
+<wire x1="-41.91" y1="-214.63" x2="-40.64" y2="-194.31" width="0" layer="19" extent="1-1"/>
+<wire x1="-19.05" y1="-128.27" x2="-40.64" y2="-194.31" width="0" layer="19" extent="1-1"/>
 <wire x1="13.97" y1="50.8" x2="-19.05" y2="-128.27" width="0" layer="19" extent="1-1"/>
 </signal>
@@
 <contactref element="Q4" pad="1"/>
 <contactref element="Q3" pad="C"/>
-<wire x1="-22.86" y1="-128.27" x2="-45.72" y2="-128.27" width="0" layer="19" extent="1-1"/>
+<wire x1="-22.86" y1="-128.27" x2="77.47" y2="21.59" width="0" layer="19" extent="1-1"/>
 <wire x1="-20.32" y1="-100.33" x2="-22.86" y2="-128.27" width="0" layer="19" extent="1-1"/>
 </signal>
-<signal name="N$21" class="2">
+<signal name="CHOPEDPOWER" class="2">
 <contactref element="L1" pad="1"/>
 <contactref element="D14" pad="C"/>
+<contactref element="T2" pad="2"/>
+<contactref element="Q1" pad="C"/>
 <contactref element="Q4" pad="2"/>
-<wire x1="-33.02" y1="-113.03" x2="-43.18" y2="-128.27" width="0" layer="19" extent="1-1"/>
+<contactref element="Q5" pad="S"/>
+<wire x1="97.79" y1="46.99" x2="-43.18" y2="-199.39" width="0" layer="19" extent="1-1"/>
+<wire x1="77.47" y1="31.75" x2="-43.18" y2="-199.39" width="0" layer="19" extent="1-1"/>
+<wire x1="77.47" y1="19.05" x2="77.47" y2="31.75" width="0" layer="19" extent="1-1"/>
+<wire x1="-33.02" y1="-113.03" x2="77.47" y2="19.05" width="0" layer="19" extent="1-1"/>
 <wire x1="-34.415" y1="-86.36" x2="-33.02" y2="-113.03" width="0" layer="19" extent="1-1"/>
 </signal>
@@
 <wire x1="-12.7" y1="-185.42" x2="-40.894" y2="-199.39" width="0" layer="19" extent="1-1"/>
 </signal>
-<signal name="B+1" class="2">
-<contactref element="D4" pad="C"/>
-</signal>
-<signal name="N$4">
-<contactref element="R3" pad="1"/>
-</signal>
-<signal name="N$2" class="2">
-<contactref element="L2" pad="1"/>
-<contactref element="D1" pad="C"/>
-<contactref element="T2" pad="2"/>
-<contactref element="Q1" pad="C"/>
-<wire x1="-45.72" y1="-179.07" x2="-43.18" y2="-199.39" width="0" layer="19" extent="1-1"/>
-<wire x1="-43.18" y1="-153.67" x2="-45.72" y2="-179.07" width="0" layer="19" extent="1-1"/>
-<wire x1="-35.685" y1="-143.51" x2="-43.18" y2="-153.67" width="0" layer="19" extent="1-1"/>
-</signal>
-<signal name="N$20" class="2">
-<contactref element="D4" pad="A"/>
-<contactref element="C13" pad="1"/>
-<contactref element="C11" pad="+"/>
-<contactref element="L2" pad="2"/>
-<wire x1="-26.67" y1="-185.42" x2="-30.48" y2="-187.96" width="0" layer="19" extent="1-1"/>
-<wire x1="-43.18" y1="-165.1" x2="-30.48" y2="-187.96" width="0" layer="19" extent="1-1"/>
-<wire x1="-27.815" y1="-143.51" x2="-43.18" y2="-165.1" width="0" layer="19" extent="1-1"/>
-</signal>
 <signal name="N$9">
 <contactref element="R3" pad="2"/>
@@
 <contactref element="T2" pad="1"/>
 <contactref element="Q1" pad="E"/>
-<wire x1="-45.72" y1="-153.67" x2="-45.466" y2="-199.39" width="0" layer="19" extent="1-1"/>
+<wire x1="77.47" y1="34.29" x2="-45.466" y2="-199.39" width="0" layer="19" extent="1-1"/>
+</signal>
+<signal name="VCC">
+<contactref element="C6" pad="+"/>
+<contactref element="U1" pad="1"/>
+<contactref element="D1" pad="A"/>
+<wire x1="-46.99" y1="-228.6" x2="-38.1" y2="-241.3" width="0" layer="19" extent="1-1"/>
+<wire x1="-44.45" y1="-214.63" x2="-46.99" y2="-228.6" width="0" layer="19" extent="1-1"/>
+</signal>
+<signal name="N$2">
+<contactref element="U1" pad="6"/>
+<contactref element="C7" pad="-"/>
+<wire x1="-44.45" y1="-234.95" x2="-39.37" y2="-207.01" width="0" layer="19" extent="1-1"/>
+</signal>
+<signal name="VB">
+<contactref element="U1" pad="8"/>
+<contactref element="C7" pad="+"/>
+<contactref element="D1" pad="C"/>
+<wire x1="-46.99" y1="-234.95" x2="-44.45" y2="-207.01" width="0" layer="19" extent="1-1"/>
+<wire x1="-45.72" y1="-241.3" x2="-46.99" y2="-234.95" width="0" layer="19" extent="1-1"/>
+</signal>
+<signal name="N$4">
+<contactref element="Q5" pad="G"/>
+<contactref element="R35" pad="2"/>
+<wire x1="97.79" y1="52.07" x2="-40.64" y2="-247.65" width="0" layer="19" extent="1-1"/>
+</signal>
+<signal name="N$20">
+<contactref element="R35" pad="1"/>
+<contactref element="U1" pad="7"/>
+<wire x1="-45.72" y1="-247.65" x2="-41.91" y2="-207.01" width="0" layer="19" extent="1-1"/>
 </signal>
 </signals>

Commit message: Simplifyed PCB with only real mosfet-driver, no charge-pump, 7805 as 5v regulator mm.
Parts:
- removed C1, C3: 100n, rcl:C050-024X044
- removed D10: 5.6v, diode:DO35Z10
- removed D2, D5: 1N4148DO35-7, diode:DO35-7
- removed Q1: BD140, transistor-power:TO126AV
- removed Q10, Q3, Q7: BD139, transistor-power:TO126AV
- removed Q4: IRF9530, transistor-fet:TO220
- removed R1: 0.033 (3W), rcl:0922/22
- removed R10: 1k, rcl:P0613V
- removed R2: 10k, rcl:0207/2V
- removed R20: 2k2, rcl:0207/2V
- removed R3, R34: 1k, rcl:0207/2V
- removed R32: 10k, rcl:P0613V
- removed R33: 680R, rcl:0207/2V
- removed R4: 330, rcl:0207/2V
- removed T1: BC547, transistor:TO92
- removed T2: TIP32, transistor:TO220
- added IC1: 7805TV, linear:TO220V
- R11: device rcl:0617/17 -> resistor:0617V
- R35: device rcl:P0613V -> rcl:0207/2V
- moved R35 319.5 mm to (86.4, 44.5)
- moved D1 312.2 mm to (74.9, 48.3), turned to 180 degrees
- moved C7 304.5 mm to (86.4, 39.4), turned to 270 degrees
- moved C6 290.5 mm to (63.5, 40.6), turned to 270 degrees
- moved U1 275.6 mm to (74.9, 39.4), turned to 270 degrees
- moved D14 178.9 mm to (86.4, 26.7), turned to 180 degrees
- moved D15 172.2 mm to (69.8, 21.6), turned to 90 degrees
- moved L1 155.7 mm to (86.4, 16.5), turned to 270 degrees
- moved C5 152.3 mm to (62.2, 14.0), turned to 180 degrees
- moved C4 130.3 mm to (55.9, 24.1), turned to 180 degrees
- moved C14 20.5 mm to (87.6, 52.1), turned to 270 degrees
- moved Q5 14.0 mm to (99.1, 35.6)
- moved BAT 11.4 mm to (68.6, 6.35)
- moved SHUNT 10.2 mm to (52.1, 6.35)
- moved R11 4.58 mm to (85.1, 59.7)
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Connections:
- removed net B-: R6.1
- removed net N$10: C1.2, Q7.C, R4.1
- removed net N$13: C1.1, D2.A, D5.C
- removed net N$19: Q3.C, Q4.1, R33.2
- removed net N$23: Q1.B, R10.2, R2.2
- removed net N$25: R10.1, T1.3
- removed net N$26: Q3.B, R32.2, R34.2
- removed net N$28: Q1.E, T2.1
- removed net N$7: D10.C, Q10.B, R20.1
- removed net N$9: R3.2, T1.2
- removed net PWM-PUMP: Q7.B
- removed net V+X2: C3.1, D2.C
- removed net VCC: C6.+, D1.A, U1.1
- net +12V: now also C6.+, D1.A, IC1.1, U1.1; no longer D5.A, Q10.C, R20.2
- net +5V: now also IC1.3; no longer Q10.E
- net B-/SHUNT: now also R6.1; no longer R1.2
- net CHARGEPWM: no longer R3.1, R34.1
- net CHOPEDPOWER: no longer Q1.C, Q4.2, T2.2
- net GND: now also IC1.2; no longer C3.2, D10.A, Q3.E, Q7.E, R1.1, R32.1, T1.1
- net V+: no longer Q4.3, R2.1, R33.1, R4.2, T2.3
Routing:
- net GND: track 0.00 -> 329.1 mm
- net +5V: track 0.00 -> 200.6 mm
- net V+: track 0.00 -> 159.3 mm, vias 0 -> 1
- net +12V: track 0.00 -> 101.0 mm
- net B-/SHUNT: track 0.00 -> 92.1 mm
- net TEMPSIGNAL: track 0.00 -> 79.9 mm
- net LED3: track 0.00 -> 70.0 mm
- net LED2: track 0.00 -> 64.2 mm, vias 0 -> 1
- net B+: track 0.00 -> 63.7 mm
- net CHARGEPWM: track 0.00 -> 61.4 mm
- net LED4: track 0.00 -> 57.6 mm, vias 0 -> 1
- net INVOLTAGESIGNAL: track 0.00 -> 51.8 mm, vias 0 -> 1
- net OUTCURRENTSIGNAL: track 0.00 -> 51.7 mm
- net N$22: track 0.00 -> 48.0 mm
- net LED5: track 0.00 -> 45.8 mm, vias 0 -> 1
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Other:
- board text added: "0.033 ohm"
