File: PCB/Smedby Charger prot.sch (EAGLE design)
At the start: 90 parts, among them IC2 TLC274D, Q1 BD140, Q10 BD139, Q2 TIP41C, Q3 BD139, Q4 IRF9530, Q7 BD139, T1 BC547, T2 TIP32

Commit message: .svn stuff removesd
Parts:
- R10: value 380 -> 1k
Other:
- note added: "12V Charger 16-20V in"
Changed lines of the file:
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@@
 <?xml version="1.0" encoding="utf-8"?>
 <!DOCTYPE eagle SYSTEM "eagle.dtd">
-<eagle version="6.4">
+<eagle version="6.5.0">
 <drawing>
 <settings>
@@
 <part name="Q3" library="transistor-power" deviceset="BD139" device=""/>
 <part name="Q4" library="transistor-fet" deviceset="IRF9530" device=""/>
-<part name="R10" library="rcl" deviceset="R-EU_" device="0613/5V" value="380"/>
+<part name="R10" library="rcl" deviceset="R-EU_" device="0613/5V" value="1k"/>
 <part name="P+3" library="supply1" deviceset="V+" device=""/>
 <part name="C11" library="rcl" deviceset="CPOL-EU" device="E7.5-18" value="1000u"/>
@@
 <text x="-33.02" y="137.16" size="1.778" layer="91">in Voltage Measure 0-66v</text>
 <text x="-76.2" y="104.14" size="1.778" layer="91">V+  +12V</text>
+<text x="101.6" y="-27.94" size="1.778" layer="91">12V Charger
+16-20V in</text>
 </plain>
 <instances>
@@
 </schematic>
 </drawing>
+<compatibility>
+<note version="6.3" minversion="6.2.2" severity="warning">
+Since Version 6.2.2 text objects can contain more than one line,
+which will not be processed correctly with this version.
+</note>
+</compatibility>
 </eagle>

Commit message: Uppdated PCB
Parts:
- removed C11: 1000u, rcl:CPOL-EUE7.5-18
- removed C13: 100n, rcl:C-EU050-024X044
- removed D4: 1N5400, diode:1N5400
- removed L2: 150uH, rcl:L-USTJ4-U1
- added C6, C7: 100u, rcl:CPOL-EUE2.5-5
- added Q5: IRF540, transistor-power:IRF540
- added R35: 100, rcl:R-EU_0613/5V
- added U1: IR2103, irf-2:IR2103
- D1: value 1N5400 -> 1N4148DO35-7; device diode:1N5400 -> diode:1N4148DO35-7
Connections:
- removed net B+1: D4.C
- removed net N$21: D14.C, L1.1, Q4.D
- new net CHOPEDPOWER: D14.C, L1.1, Q1.C, Q4.D, Q5.S, T2.C
- new net VB: C7.+, D1.C, U1.VB
- new net VCC: C6.+, D1.A, U1.VCC
- net CHARGEPWM: now also R3.1, U1.HIN
- net GND: now also C6.-, U1./LIN, U1.COM; no longer C11.-, C13.2, D1.A
- net N$2: now also C7.-, U1.VS; no longer D1.C, L2.1, Q1.C, T2.C
- net N$20: now also R35.1, U1.HO; no longer C11.+, C13.1, D4.A, L2.2
- net N$4: now also Q5.G, R35.2; no longer R3.1
- net V+: now also Q5.D
Other:
- note added: "Simple P-Fet driver"
- moved on the sheet: C4, C5, D14, D15, L1

Commit message: Simplifyed PCB with only real mosfet-driver, no charge-pump, 7805 as 5v regulator mm.
Parts:
- removed C1, C3: 100n, rcl:C-EU050-024X044
- removed D10: 5.6v, diode:BZX55
- removed D2, D5: 1N4148DO35-7, diode:1N4148DO35-7
- removed Q1: BD140, transistor-power:BD140
- removed Q10, Q3, Q7: BD139, transistor-power:BD139
- removed Q4: IRF9530, transistor-fet:IRF9530
- removed R1: 0.033 (3W), rcl:R-EU_0922/22
- removed R10: 1k, rcl:R-EU_0613/5V
- removed R2: 10k, rcl:R-EU_0207/2V
- removed R20: 2k2, rcl:R-EU_0207/2V
- removed R3, R34: 1k, rcl:R-EU_0207/2V
- removed R32: 10k, rcl:R-EU_0613/5V
- removed R33: 680R, rcl:R-EU_0207/2V
- removed R4: 330, rcl:R-EU_0207/2V
- removed T1: BC547, transistor:BC547
- removed T2: TIP32, transistor:TIP32
- added IC1: 7805TV, linear:7805TV
- R11: device rcl:R-EU_0617/17 -> resistor:R-EU_0617/5V
- R35: device rcl:R-EU_0613/5V -> rcl:R-EU_0207/2V
Connections:
- removed net B-: R6.1
- removed net N$10: C1.2, Q7.C, R4.1
- removed net N$13: C1.1, D2.A, D5.C
- removed net N$19: Q3.C, Q4.G, R33.2
- removed net N$23: Q1.B, R10.2, R2.2
- removed net N$25: R10.1, T1.C
- removed net N$26: Q3.B, R32.2, R34.2
- removed net N$28: Q1.E, T2.B
- removed net N$7: D10.C, Q10.B, R20.1
- removed net N$9: R3.2, T1.B
- removed net PWM-PUMP: Q7.B
- removed net V+X2: C3.1, D2.C
- removed net VCC: C6.+, D1.A, U1.VCC
- net +12V: now also C6.+, D1.A, IC1.VI, U1.VCC; no longer D5.A, Q10.C, R20.2
- net +5V: now also IC1.VO; no longer Q10.E
- net B-/SHUNT: now also R6.1; no longer R1.2
- net CHARGEPWM: no longer R3.1, R34.1
- net CHOPEDPOWER: no longer Q1.C, Q4.D, T2.C
- net GND: now also IC1.GND; no longer C3.2, D10.A, Q3.E, Q7.E, R1.1, R32.1, T1.E
- net V+: no longer Q4.S, R2.1, R33.1, R4.2, T2.E
Other:
- note removed: "12V Charger 16-20V in"
- note removed: "Simple P-Fet driver"
- note removed: "V+ +12V"
- moved on the sheet: C4, C5, C6, C7, D1, D14, D15, L1, Q5, R35, U1
